File: peacock_tail_brd.kicad_sch (KiCad schematic)
At the start: 27 parts, among them J1 Conn_01x03, J10 Screw_Terminal_01x02, J2 Conn_01x03, J3 Conn_01x03, J4 Conn_01x03, J5 Conn_01x03, J7 Conn_01x04, J8 Conn_01x04, U1 RP2040-ZERO, U2 L7805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

Commit message: lm2596 update
Signed-off-by: Sezgin AÇIKGÖZ <sacikgoz@tarla-fel.org>
Parts:
- removed C1: 0.33uF/50V, PCM_Capacitor_SMD_AKL:C_0805_2012Metric, symbol PCM_Capacitor_AKL:C_0805
- removed C2: 0.1uF/50V, PCM_Capacitor_SMD_AKL:C_0805_2012Metric, symbol PCM_Capacitor_AKL:C_0805
- removed U2: L7805, Package_TO_SOT_THT:TO-220-3_Vertical, symbol Regulator_Linear:L7805
- added C1: 100uF, PCM_Capacitor_SMD_AKL:CP_Elec_6.3x7.7, symbol Device:C_Polarized
- added C2, C6: 100nF, Capacitor_SMD:C_0603_1608Metric, symbol Device:C
- added C5: 220uF/10V, PCM_Capacitor_SMD_AKL:CP_Elec_6.3x7.7, symbol Device:C_Polarized
- added D1: SS34, Diode_SMD:D_SMA, symbol Diode:SS34
- added D2: LED, LED_SMD:LED_0603_1608Metric, symbol Device:LED
- added L1: 47uH, Inductor_SMD:L_Bourns_SRR1208_12.7x12.7mm, symbol Device:L
- added R5: 1K, Resistor_SMD:R_0603_1608Metric, symbol Device:R
- added R6: 4K7, Resistor_SMD:R_0603_1608Metric, symbol Device:R
- added RV1: 10K, Potentiometer_THT:Potentiometer_Bourns_3296W_Vertical, symbol Device:R_Potentiometer
- added U2: LM2596S-ADJ, Package_TO_SOT_SMD:TO-263-5_TabPin3, symbol Regulator_Switching:LM2596S-ADJ
- renumbered J10 to J6
Connections:
- net +5V: now also C5.1, C6.1, L1.2, R6.1, RV1.1
- net GND: now also C1.2, C2.2, C5.2, C6.2, D1.2 (A), D2.1 (K), R5.2, U2.3 (GND), U2.5 (~{ON}/OFF)
- net VDC renamed VIN
- net VIN: now also C1.1, C2.1, U2.1 (VIN)
- new net: R5.1, RV1.2, RV1.3, U2.4 (FB)
- new net: D2.2 (A), R6.2
- new net SW: D1.1 (K), L1.1, U2.2 (OUT)
Other:
- moved on the sheet: J6, U1
